File: nofly.kicad_pcb (KiCad board)
At the start: 4 copper layers, 23.6 x 8.3 mm, 8 parts, among them J1 USB_C_Receptacle_USB2.0_16P, J2 Conn_01x04, U1 USBLC6-2P6

Commit message: Update component metadata
Parts:
- F1: value ASMD0805H050 -> SMD0805-050
- J1: value USB_C_Receptacle_USB2.0_16P -> TYPE-C-31-M-12
- J2: value Conn_01x04 -> 781710004
Connections:
- H1 pad 1: (no net) -> GND
Changed lines of the file:
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@@
 			(layers "*.Cu" "*.Mask")
 			(remove_unused_layers no)
+			(net 5 "GND")
+			(pinfunction "MP")
+			(pintype "input")
 			(zone_connect 2)
 		)
@@
 			)
 		)
-		(property "Value" "USB_C_Receptacle_USB2.0_16P"
+		(property "Value" "TYPE-C-31-M-12"
 			(at 0.05 7.35 0)
 			(layer "F.Fab")
@@
 				(font
 					(size 1.27 1.27)
+					(thickness 0.15)
+				)
+			)
+		)
+		(property "Manufacturer" "Koren Hroparts"
+			(at 0 0 180)
+			(unlocked yes)
+			(layer "F.Fab")
+			(hide yes)
+			(effects
+				(font
+					(size 1 1)
+					(thickness 0.15)
+				)
+			)
+		)
+		(property "Manufacturer Part Number" "TYPE-C-31-M-12 "
+			(at 0 0 180)
+			(unlocked yes)
+			(layer "F.Fab")
+			(hide yes)
+			(effects
+				(font
+					(size 1 1)
+					(thickness 0.15)
+				)
+			)
+		)
+		(property "LCSC Part Number" "C165948"
+			(at 0 0 180)
+			(unlocked yes)
+			(layer "F.Fab")
+			(hide yes)
+			(effects
+				(font
+					(size 1 1)
+					(thickness 0.15)
+				)
+			)
+		)
+		(property "Package" ""
+			(at 0 0 180)
+			(unlocked yes)
+			(layer "F.Fab")
+			(hide yes)
+			(effects
+				(font
+					(size 1 1)
 					(thickness 0.15)
 				)
@@
 		)
 		(property "Value" "USBLC6-2P6"
-			(at 0 -1.75 180)
-			(layer "B.Fab")
-			(effects
-				(font
-					(size 1 1)
-					(thickness 0.15)
+			(at 0 -1.35 180)
+			(layer "B.Fab")
+			(effects
+				(font
+					(size 0.5 0.5)
+					(thickness 0.1)
+					(bold yes)
 				)
 				(justify mirror)
@@
 				(font
 					(size 1.27 1.27)
+					(thickness 0.15)
+				)
+				(justify mirror)
+			)
+		)
+		(property "Manufacturer" "STMicroelectronics"
+			(at 0 0 0)
+			(unlocked yes)
+			(layer "B.Fab")
+			(hide yes)
+			(effects
+				(font
+					(size 1 1)
+					(thickness 0.15)
+				)
+				(justify mirror)
+			)
+		)
+		(property "Manufacturer Part Number" "USBLC6-2P6"
+			(at 0 0 0)
+			(unlocked yes)
+			(layer "B.Fab")
+			(hide yes)
+			(effects
+				(font
+					(size 1 1)
+					(thickness 0.15)
+				)
+				(justify mirror)
+			)
+		)
+		(property "LCSC Part Number" "C15999"
+			(at 0 0 0)
+			(unlocked yes)
+			(layer "B.Fab")
+			(hide yes)
+			(effects
+				(font
+					(size 1 1)
+					(thickness 0.15)
+				)
+				(justify mirror)
+			)
+		)
+		(property "Package" "SOT-666"
+			(at 0 0 0)
+			(unlocked yes)
+			(layer "B.Fab")
+			(hide yes)
+			(effects
+				(font
+					(size 1 1)
 					(thickness 0.15)
 				)
@@
 			)
 		)
-		(property "Value" "Conn_01x04"
+		(property "Value" "781710004"
 			(at 0 -1 0)
 			(unlocked yes)
@@
 				(font
 					(size 1.27 1.27)
+					(thickness 0.15)
+				)
+				(justify mirror)
+			)
+		)
+		(property "Manufacturer" "MOLEX"
+			(at 0 0 180)
+			(unlocked yes)
+			(layer "B.Fab")
+			(hide yes)
+			(effects
+				(font
+					(size 1 1)
+					(thickness 0.15)
+				)
+				(justify mirror)
+			)
+		)
+		(property "Manufacturer Part Number" "781710004"
+			(at 0 0 180)
+			(unlocked yes)
+			(layer "B.Fab")
+			(hide yes)
+			(effects
+				(font
+					(size 1 1)
+					(thickness 0.15)
+				)
+				(justify mirror)
+			)
+		)
+		(property "LCSC Part Number" "C588524"
+			(at 0 0 180)
+			(unlocked yes)
+			(layer "B.Fab")
+			(hide yes)
+			(effects
+				(font
+					(size 1 1)
+					(thickness 0.15)
+				)
+				(justify mirror)
+			)
+		)
+		(property "Package" ""
+			(at 0 0 180)
+			(unlocked yes)
+			(layer "B.Fab")
+			(hide yes)
+			(effects
+				(font
+					(size 1 1)
 					(thickness 0.15)
 				)
@@
 		)
 		(property "Value" "5.1k"
-			(at 0 -1.17 90)
-			(layer "B.Fab")
-			(effects
-				(font
-					(size 1 1)
-					(thickness 0.15)
+			(at 0 -0.79 90)
+			(layer "B.Fab")
+			(effects
+				(font
+					(size 0.5 0.5)
+					(thickness 0.1)
+					(bold yes)
 				)
 				(justify mirror)
@@
 		)
 		(property "Value" "5.1k"
-			(at 0 -1.17 90)
-			(layer "B.Fab")
-			(effects
-				(font
-					(size 1 1)
-					(thickness 0.15)
+			(at 0 -1 90)
+			(layer "B.Fab")
+			(effects
+				(font
+					(size 0.5 0.5)
+					(thickness 0.1)
+					(bold yes)
 				)
 				(justify mirror)
@@
 			)
 		)
-		(property "Value" "ASMD0805H050"
-			(at 0 -1.65 90)
-			(layer "B.Fab")
-			(effects
-				(font
-					(size 1 1)
-					(thickness 0.15)
+		(property "Value" "SMD0805-050"
+			(at -0.0125 -1.350003 90)
+			(layer "B.Fab")
+			(effects
+				(font
+					(size 0.5 0.5)
+					(thickness 0.1)
+					(bold yes)
 				)
 				(justify mirror)
@@
 			)
 		)
-		(property "Manufacturer" "Shenzhen JDT Fuse"
+		(property "Manufacturer" "TECHFUSE"
 			(at 0 0 270)
 			(unlocked yes)
@@
 			)
 		)
-		(property "Manufacturer Part Number" "ASMD0805H050"
+		(property "Manufacturer Part Number" "SMD0805-050 "
 			(at 0 0 270)
 			(unlocked yes)
@@
 			)
 		)
-		(property "LCSC Part Number" "C48783086"
+		(property "LCSC Part Number" "C66452"
 			(at 0 0 270)
 			(unlocked yes)
