File: nofly.kicad_pcb (KiCad board)
At the start: 4 copper layers, 23.6 x 8.3 mm, 8 parts, among them J1 TYPE-C-31-M-12, J2 781710004, U1 USBLC6-2P6

Commit message: Finish wiring... Maybe?
Parts:
- moved R1 13.0 mm to (141.4, 69.5), turned to -90 degrees
- moved F1 1.24 mm to (141.5, 66.2)
- moved R2 0.71 mm to (129.1, 67.9)
Routing:
- net D+: track 8.48 -> 14.9 mm, vias 2 -> 3
- net D-: track 8.50 -> 14.6 mm, vias 2 -> 3
- net Net-(J1-CC1): track 11.6 -> 6.70 mm, vias 2 -> 1
- net VBUS: track 21.4 -> 22.4 mm
- net 5V: track 5.23 -> 4.71 mm
- net Net-(J1-CC2): track 7.38 -> 7.52 mm, vias 2 -> 1
- net GND: vias 0 -> 2

Commit message: Finish wiring now?
Parts:
- J2: value 781710004 -> Conn_01x04_MountingPin; footprint acheron_Connectors:MOLEX_781710004 -> acheron_Connectors:MOLEX_PicoEZMate_781710004
Connections:
- J2 pad MP: (no net) -> GND
Routing:
- net VBUS: track 22.4 -> 24.9 mm
- net D+: track 14.9 -> 13.3 mm
- net D-: track 14.6 -> 13.2 mm
- net GND: vias 2 -> 3

Commit message: Some rerouting and checks
Parts:
- moved F1 0.07 mm to (141.5, 66.2)
Routing:
- net VBUS: track 24.9 -> 24.0 mm
Other:
- board text added: "V 1.0"
- board text removed: "REV. A"
Changed lines of the file:
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@@
 		(capping no)
 		(filling no)
-		(grid_origin 137.494001 66.829998)
+		(grid_origin 147.8 62.4)
 		(pcbplotparams
 			(layerselection 0x00000000_00000000_55555555_5755f5ff)
@@
 	(footprint "Fuse:Fuse_0805_2012Metric"
 		(layer "B.Cu")
-		(at 141.549997 66.177 -90)
+		(at 141.489997 66.2195 -90)
 		(descr "Fuse SMD 0805 (2012 Metric), square (rectangular) end terminal, IPC-7351 nominal, (Body size source: https://docs.google.com/spreadsheets/d/1BsfQQcO9C6DZCsRaXUlFlo91Tg2WpOkGARC1WS5S8t0/edit?usp=sharing), generated with kicad-footprint-generator")
 		(tags "fuse")
@@
 		(layer "Edge.Cuts")
 	)
-	(gr_text "REV. A"
+	(gr_text "V 1.0"
 		(at 128.9 67.4 270)
 		(layer "F.SilkS")
@@
 	)
 	(via
-		(at 141.544781 64.13617)
+		(at 141.484781 64.582)
 		(size 0.6)
 		(drill 0.3)
@@
 	)
 	(segment
-		(start 141.549997 64.141386)
-		(end 141.544781 64.13617)
+		(start 141.484781 65.276784)
+		(end 141.489997 65.282)
 		(width 0.2)
 		(layer "B.Cu")
@@
 	)
 	(segment
-		(start 141.549997 65.2395)
-		(end 141.549997 64.141386)
+		(start 141.484781 64.582)
+		(end 141.484781 65.276784)
 		(width 0.5)
 		(layer "B.Cu")
@@
 	)
 	(segment
-		(start 141.544781 66.789222)
-		(end 141.544781 64.13617)
-		(width 0.5)
-		(layer "In2.Cu")
-		(net "VBUS")
-	)
-	(segment
 		(start 132.315135 67.567168)
 		(end 133.747651 66.134652)
@@
 	)
 	(segment
+		(start 141.484781 64.582)
+		(end 141.484781 66.849222)
+		(width 0.5)
+		(layer "In2.Cu")
+		(net "VBUS")
+	)
+	(segment
 		(start 140.621004 67.712999)
-		(end 141.544781 66.789222)
+		(end 141.484781 66.849222)
 		(width 0.5)
 		(layer "In2.Cu")
@@
 	)
 	(segment
-		(start 141.437497 67.002)
-		(end 141.549997 67.1145)
-		(width 0.5)
-		(layer "B.Cu")
-		(net "5V")
-	)
-	(segment
-		(start 139.124365 67.002)
-		(end 141.437497 67.002)
+		(start 138.597365 66.475)
+		(end 137.099997 66.475)
 		(width 0.5)
 		(layer "B.Cu")
@@
 	)
 	(segment
-		(start 138.597365 66.475)
-		(end 139.124365 67.002)
+		(start 141.489997 67.157)
+		(end 139.279365 67.157)
 		(width 0.5)
 		(layer "B.Cu")
@@
 	)
 	(segment
-		(start 137.099997 66.475)
+		(start 139.279365 67.157)
 		(end 138.597365 66.475)
 		(width 0.5)

Commit message: Remove visible silkscreen designators
Parts:
- J2: value Conn_01x04_MountingPin -> 781710004 / M1201RS-04-BK
- U1: footprint Package_TO_SOT_SMD:SOT-666 -> Package_TO_SOT_SMD:SOT-563
Changed lines of the file:
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@@
 		(capping no)
 		(filling no)
-		(grid_origin 147.8 62.4)
+		(aux_axis_origin 135.299997 66.475)
+		(grid_origin 135.299997 64.55)
 		(pcbplotparams
-			(layerselection 0x00000000_00000000_55555555_5755f5ff)
+			(layerselection 0x00000000_00000000_5555555f_5755f5ff)
 			(plot_on_all_layers_selection 0x00000000_00000000_00000000_00000000)
 			(disableapertmacros no)
@@
 			(usegerberattributes yes)
 			(usegerberadvancedattributes yes)
-			(creategerberjobfile yes)
+			(creategerberjobfile no)
 			(dashed_line_dash_ratio 12)
 			(dashed_line_gap_ratio 3)
@@
 			(plotframeref no)
 			(mode 1)
-			(useauxorigin no)
+			(useauxorigin yes)
 			(pdf_front_fp_property_popups yes)
 			(pdf_back_fp_property_popups yes)
@@
 			(outputformat 1)
 			(mirror no)
-			(drillshape 1)
+			(drillshape 0)
 			(scaleselection 1)
-			(outputdirectory "")
+			(outputdirectory "../release/gerbers")
 		)
 	)
@@
 		)
 	)
-	(footprint "Package_TO_SOT_SMD:SOT-666"
+	(footprint "Package_TO_SOT_SMD:SOT-563"
 		(layer "B.Cu")
 		(at 135.299997 64.55)
-		(descr "SOT666")
-		(tags "SOT-666")
+		(descr "SOT, 6 Pin (https://www.jedec.org/system/files/docs/MO-293B.pdf)")
+		(tags "SOT TO_SOT_SMD JEDEC-MO-293-UAAD Texas-DRL-6")
 		(property "Reference" "U1"
-			(at 0 2.000001 180)
+			(at -1.4 0 180)
 			(layer "B.SilkS")
 			(hide yes)
@@
 				(font
 					(size 1 1)
-					(thickness 0.15)
+					(thickness 0.2)
+					(bold yes)
 				)
-				(justify mirror)
+				(justify left mirror)
 			)
 		)
 		(property "Value" "USBLC6-2P6"
-			(at 0 -1.35 180)
+			(at 0 -1.65 180)
 			(layer "B.Fab")
 			(effects
 				(font
-					(size 0.5 0.5)
-					(thickness 0.1)
+					(size 0.3 0.3)
+					(thickness 0.06)
 					(bold yes)
 				)
@@
 		(property "Datasheet" "https://www.st.com/resource/en/datasheet/usblc6-2.pdf"
 			(at 0 0 180)
-			(unlocked yes)
 			(layer "B.Fab")
 			(hide yes)
@@
 				(font
 					(size 1.27 1.27)
-					(thickness 0.15)
 				)
 				(justify mirror)
@@
 		(property "Description" "Very low capacitance ESD protection diode, 2 data-line, SOT-666"
 			(at 0 0 180)
-			(unlocked yes)
 			(layer "B.Fab")
 			(hide yes)
@@
 				(font
 					(size 1.27 1.27)
+				)
+				(justify mirror)
+			)
+		)
+		(property "KiLib_Generator" "package/gullwing"
+			(at 0 0 180)
+			(layer "B.SilkS")
+			(hide yes)
+			(effects
+				(font
+					(size 1 1)
 					(thickness 0.15)
 				)
@@
 			)
 		)
-		(property "Manufacturer" "STMicroelectronics"
+		(property "Manufacturer" "YTL"
 			(at 0 0 0)
 			(unlocked yes)
@@
 			)
 		)
-		(property "LCSC Part Number" "C15999"
+		(property "LCSC Part Number" "C53059594"
 			(at 0 0 0)
 			(unlocked yes)
@@
 		(sheetname "/")
 		(sheetfile "nofly.kicad_sch")
-		(units
-			(unit
-				(name "A")
-				(pins "1" "3" "5" "2" "6" "4")
-			)
-		)
 		(attr smd)
 		(duplicate_pad_numbers_are_jumpers no)
 		(fp_line
-			(start 0.65 -0.99)
-			(end -0.65 -0.99)
+			(start -0.425568 0.935)
+			(end 0.71 0.935)
 			(stroke
 				(width 0.12)
@@
 		)
 		(fp_line
-			(start 0.65 0.99)
-			(end -0.4 0.99)
+			(start 0.71 -0.935)
+			(end -0.71 -0.935)
 			(stroke
 				(width 0.12)
@@
 		(fp_poly
 			(pts
-				(xy -1.866 0.7915) (xy -1.358 0.5375) (xy -1.866 0.2835)
+				(xy -1.3125 0.5) (xy -1.5025 0.36) (xy -1.5025 0.64)
 			)
 			(stroke
@@
 		)
 		(fp_line
-			(start -1.5 -1.1)
-			(end 1.5 -1.1)
+			(start -1.2 -0.83)
+			(end -1.2 0.83)
 			(stroke
 				(width 0.05)
@@
 		)
 		(fp_line
-			(start -1.5 1.1)
-			(end -1.5 -1.1)
+			(start -1.2 0.83)
+			(end -0.75 0.83)
 			(stroke
 				(width 0.05)
@@
 		)
 		(fp_line
-			(start -1.5 1.1)
-			(end 1.5 1.1)
+			(start -0.75 -0.95)
+			(end -0.75 -0.83)
 			(stroke
 				(width 0.05)
@@
 		)
 		(fp_line
-			(start 1.5 -1.1)
-			(end 1.5 1.1)
+			(start -0.75 -0.83)
+			(end -1.2 -0.83)
 			(stroke
 				(width 0.05)
@@
 		)
 		(fp_line
-			(start -0.65 0.53)
-			(end -0.65 -0.85)
+			(start -0.75 0.83)
+			(end -0.75 0.95)
 			(stroke
-				(width 0.1)
+				(width 0.05)
 				(type solid)
 			)
-			(layer "B.Fab")
+			(layer "B.CrtYd")
 		)
 		(fp_line
-			(start -0.65 0.53)
-			(end -0.33 0.85)
+			(start -0.75 0.95)
+			(end 0.75 0.95)
 			(stroke
-				(width 0.1)
+				(width 0.05)
 				(type solid)
 			)
-			(layer "B.Fab")
+			(layer "B.CrtYd")
 		)
 		(fp_line
-			(start 0.65 -0.85)
-			(end -0.65 -0.85)
+			(start 0.75 -0.95)
+			(end -0.75 -0.95)
 			(stroke
-				(width 0.1)
+				(width 0.05)
 				(type solid)
 			)
-			(layer "B.Fab")
+			(layer "B.CrtYd")
 		)
 		(fp_line
-			(start 0.65 0.85)
-			(end -0.33 0.85)
+			(start 0.75 -0.83)
+			(end 0.75 -0.95)
 			(stroke
-				(width 0.1)
+				(width 0.05)
 				(type solid)
 			)
-			(layer "B.Fab")
+			(layer "B.CrtYd")
 		)
 		(fp_line
-			(start 0.65 0.85)
-			(end -0.33 0.85)
+			(start 0.75 0.83)
+			(end 1.2 0.83)
 			(stroke
-				(width 0.1)
+				(width 0.05)
 				(type solid)
 			)
-			(layer "B.Fab")
+			(layer "B.CrtYd")
+		)
+		(fp_line
+			(start 0.75 0.95)
+			(end 0.75 0.83)
+			(stroke
+				(width 0.05)
+				(type solid)
+			)
+			(layer "B.CrtYd")
+		)
+		(fp_line
+			(start 1.2 -0.83)
+			(end 0.75 -0.83)
+			(stroke
+				(width 0.05)
+				(type solid)
+			)
+			(layer "B.CrtYd")
 		)
 		(fp_line
-			(start 0.65 0.85)
-			(end 0.65 -0.85)
+			(start 1.2 0.83)
+			(end 1.2 -0.83)
+			(stroke
+				(width 0.05)
+				(type solid)
+			)
+			(layer "B.CrtYd")
+		)
+		(fp_poly
+			(pts
+				(xy -0.3 0.8) (xy 0.6 0.8) (xy 0.6 -0.8) (xy -0.6 -0.8) (xy -0.6 0.5)
+			)
 			(stroke
 				(width 0.1)
 				(type solid)
 			)
+			(fill no)
 			(layer "B.Fab")
 		)
@@
 			(effects
 				(font
-					(size 0.5 0.5)
-					(thickness 0.075)
+					(size 0.4 0.4)
+					(thickness 0.06)
 				)
 				(justify mirror)
@@
 		)
 		(pad "1" smd roundrect
-			(at -0.85 0.5375)
-			(size 0.5 0.375)
+			(at -0.7125 0.5)
+			(size 0.675 0.35)
 			(layers "B.Cu" "B.Mask" "B.Paste")
 			(roundrect_rratio 0.25)
@@
 		)
 		(pad "2" smd roundrect
-			(at -0.925 0)
-			(size 0.65 0.3)
+			(at -0.7125 0)
+			(size 0.675 0.35)
 			(layers "B.Cu" "B.Mask" "B.Paste")
 			(roundrect_rratio 0.25)
@@
 			(pinfunction "GND_2")
 			(pintype "passive")
-			(zone_connect 2)
 		)
 		(pad "3" smd roundrect
-			(at -0.85 -0.5375)
-			(size 0.5 0.375)
+			(at -0.7125 -0.5)
+			(size 0.675 0.35)
 			(layers "B.Cu" "B.Mask" "B.Paste")
 			(roundrect_rratio 0.25)
@@
 		)
 		(pad "4" smd roundrect
-			(at 0.85 -0.5375)
-			(size 0.5 0.375)
+			(at 0.7125 -0.5)
+			(size 0.675 0.35)
 			(layers "B.Cu" "B.Mask" "B.Paste")
 			(roundrect_rratio 0.25)
@@
 		)
 		(pad "5" smd roundrect
-			(at 0.925 0)
-			(size 0.65 0.3)
+			(at 0.7125 0)
+			(size 0.675 0.35)
 			(layers "B.Cu" "B.Mask" "B.Paste")
 			(roundrect_rratio 0.25)
@@
 		)
 		(pad "6" smd roundrect
-			(at 0.85 0.5375)
-			(size 0.5 0.375)
+			(at 0.7125 0.5)
+			(size 0.675 0.35)
 			(layers "B.Cu" "B.Mask" "B.Paste")
 			(roundrect_rratio 0.25)
@@
 		)
 		(embedded_fonts no)
-		(model "${KICAD9_3DMODEL_DIR}/Package_TO_SOT_SMD.3dshapes/SOT-666.step"
+		(model "${KICAD10_3DMODEL_DIR}/Package_TO_SOT_SMD.3dshapes/SOT-563.step"
 			(offset
 				(xyz 0 0 0)
@@
 			)
 		)
-		(property "Value" "Conn_01x04_MountingPin"
+		(property "Value" "781710004 / M1201RS-04-BK"
 			(at 0 -1 0)
 			(unlocked yes)
@@
 			)
 		)
-		(property "Manufacturer" "MOLEX"
+		(property "Manufacturer" "XFCN"
 			(at 0 0 180)
 			(unlocked yes)
@@
 			)
 		)
-		(property "LCSC Part Number" "C588524"
+		(property "LCSC Part Number" "C2840019"
 			(at 0 0 180)
 			(unlocked yes)
@@
 		)
 		(property "Value" "SMD0805-050"
-			(at -0.0125 -1.350003 90)
+			(at -0.0125 0.889997 90)
 			(layer "B.Fab")
 			(effects
 				(font
-					(size 0.5 0.5)
-					(thickness 0.1)
+					(size 0.3 0.3)
+					(thickness 0.06)
 					(bold yes)
 				)
@@
 		)
 	)
+	(point
+		(at 135.299997 66.475)
+		(size 1)
+		(layer "B.Cu")
+	)
 	(via
 		(at 135.294001 64.102999)
@@
 	)
 	(segment
+		(start 139.124364 67.002)
+		(end 138.597365 66.475)
+		(width 0.5)
+		(layer "B.Cu")
+		(net "5V")
+	)
+	(segment
 		(start 141.489997 67.157)
-		(end 139.279365 67.157)
+		(end 141.334997 67.002)
 		(width 0.5)
 		(layer "B.Cu")
@@
 	)
 	(segment
-		(start 139.279365 67.157)
-		(end 138.597365 66.475)
+		(start 141.334997 67.002)
+		(end 139.124364 67.002)
 		(width 0.5)
 		(layer "B.Cu")

Commit message: Rotate ESD chip for clearance
Parts:
- moved U1 0.23 mm to (135.3, 64.8), turned to 90 degrees
Connections:
- U1 pad 1: DO+ -> DO-
- U1 pad 3: D+ -> DO+
- U1 pad 4: D- -> D+
- U1 pad 6: DO- -> D-
Routing:
- net VBUS: track 24.0 -> 31.0 mm
- net D+: track 13.3 -> 16.4 mm
- net Net-(J1-CC1): track 6.70 -> 9.19 mm
- net D-: track 13.2 -> 12.1 mm
- net Net-(J1-CC2): track 7.28 -> 8.30 mm
