File: nofly.kicad_sch (KiCad schematic)
At the start: 8 parts, among them J1 USB_C_Receptacle_USB2.0_16P, J2 Conn_01x04, U1 USBLC6-2P6

Commit message: Organize schematic
Other:
- note added: "EZM"
- note added: "MOUNTING"
- note added: "PROTECTION"
- note added: "USB"
- moved on the sheet: F1, H1, H2, J1, J2, R1, R2, U1

Commit message: Update component metadata
Parts:
- F1: value ASMD0805H050 -> SMD0805-050; LCSC Part Number C48783086 -> C66452; Manufacturer Shenzhen JDT Fuse -> TECHFUSE; Manufacturer Part Number ASMD0805H050 -> SMD0805-050
- J1: value USB_C_Receptacle_USB2.0_16P -> TYPE-C-31-M-12; LCSC Part Number (none) -> C165948; Manufacturer (none) -> Koren Hroparts; Manufacturer Part Number (none) -> TYPE-C-31-M-12
- J2: value Conn_01x04 -> 781710004; LCSC Part Number (none) -> C588524; Manufacturer (none) -> MOLEX; Manufacturer Part Number (none) -> 781710004
- U1: LCSC Part Number (none) -> C15999; Manufacturer (none) -> STMicroelectronics; Manufacturer Part Number (none) -> USBLC6-2P6; Package (none) -> SOT-666
Connections:
- net GND: now also H1.1 (MP); no longer H1.MP
Changed lines of the file:
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@@
-	(wire
-		(pts
-			(xy 38.1 41.91) (xy 38.1 44.45)
-		)
-		(stroke
-			(width 0)
-			(type default)
-		)
-	)
 	(wire
 		(pts
@@
 			)
 		)
-		(property "Value" "ASMD0805H050"
+		(property "Value" "SMD0805-050"
 			(at 184.15 67.0814 90)
 			(effects
@@
 			)
 		)
-		(property "Manufacturer" "Shenzhen JDT Fuse"
+		(property "Manufacturer" "TECHFUSE"
 			(at 184.15 69.85 90)
 			(effects
@@
 			)
 		)
-		(property "Manufacturer Part Number" "ASMD0805H050"
+		(property "Manufacturer Part Number" "SMD0805-050 "
 			(at 184.15 69.85 90)
 			(effects
@@
 			)
 		)
-		(property "LCSC Part Number" "C48783086"
+		(property "LCSC Part Number" "C66452"
 			(at 184.15 69.85 90)
 			(effects
@@
 			)
 		)
+		(property "Manufacturer" "STMicroelectronics"
+			(at 184.15 43.18 0)
+			(effects
+				(font
+					(size 1.27 1.27)
+				)
+				(hide yes)
+			)
+		)
+		(property "Manufacturer Part Number" "USBLC6-2P6"
+			(at 184.15 43.18 0)
+			(effects
+				(font
+					(size 1.27 1.27)
+				)
+				(hide yes)
+			)
+		)
+		(property "LCSC Part Number" "C15999"
+			(at 184.15 43.18 0)
+			(effects
+				(font
+					(size 1.27 1.27)
+				)
+				(hide yes)
+			)
+		)
+		(property "Package" "SOT-666"
+			(at 184.15 43.18 0)
+			(effects
+				(font
+					(size 1.27 1.27)
+				)
+				(hide yes)
+			)
+		)
 		(pin "4"
 		)
@@
 	(symbol
 		(lib_id "power:GND")
-		(at 38.1 44.45 0)
+		(at 38.1 41.91 0)
 		(unit 1)
 		(exclude_from_sim no)
@@
 		(fields_autoplaced yes)
 		(property "Reference" "#PWR01"
-			(at 38.1 50.8 0)
+			(at 38.1 48.26 0)
 			(effects
 				(font
@@
 		)
 		(property "Value" "GND"
-			(at 38.1 49.53 0)
+			(at 38.1 46.99 0)
 			(effects
 				(font
@@
 		)
 		(property "Footprint" ""
-			(at 38.1 44.45 0)
+			(at 38.1 41.91 0)
 			(effects
 				(font
@@
 		)
 		(property "Datasheet" ""
-			(at 38.1 44.45 0)
+			(at 38.1 41.91 0)
 			(effects
 				(font
@@
 		)
 		(property "Description" "Power symbol creates a global label with name \"GND\" , ground"
-			(at 38.1 44.45 0)
+			(at 38.1 41.91 0)
 			(effects
 				(font
@@
 			)
 		)
-		(property "Value" "USB_C_Receptacle_USB2.0_16P"
+		(property "Value" "TYPE-C-31-M-12"
 			(at 111.76 29.21 0)
 			(effects
@@
 		)
 		(property "Description" "USB 2.0-only 16P Type-C Receptacle connector"
+			(at 111.76 48.895 0)
+			(effects
+				(font
+					(size 1.27 1.27)
+				)
+				(hide yes)
+			)
+		)
+		(property "Manufacturer" "Koren Hroparts"
+			(at 111.76 48.895 0)
+			(effects
+				(font
+					(size 1.27 1.27)
+				)
+				(hide yes)
+			)
+		)
+		(property "Manufacturer Part Number" "TYPE-C-31-M-12 "
+			(at 111.76 48.895 0)
+			(effects
+				(font
+					(size 1.27 1.27)
+				)
+				(hide yes)
+			)
+		)
+		(property "LCSC Part Number" "C165948"
+			(at 111.76 48.895 0)
+			(effects
+				(font
+					(size 1.27 1.27)
+				)
+				(hide yes)
+			)
+		)
+		(property "Package" ""
 			(at 111.76 48.895 0)
 			(effects
@@
 			)
 		)
-		(property "Value" "Conn_01x04"
+		(property "Value" "781710004"
 			(at 250.19 39.3699 0)
 			(effects
@@
 		)
 		(property "Description" "Generic connector, single row, 01x04, script generated (kicad-library-utils/schlib/autogen/connector/)"
+			(at 247.65 36.83 0)
+			(effects
+				(font
+					(size 1.27 1.27)
+				)
+				(hide yes)
+			)
+		)
+		(property "Manufacturer" "MOLEX"
+			(at 247.65 36.83 0)
+			(effects
+				(font
+					(size 1.27 1.27)
+				)
+				(hide yes)
+			)
+		)
+		(property "Manufacturer Part Number" "781710004"
+			(at 247.65 36.83 0)
+			(effects
+				(font
+					(size 1.27 1.27)
+				)
+				(hide yes)
+			)
+		)
+		(property "LCSC Part Number" "C588524"
+			(at 247.65 36.83 0)
+			(effects
+				(font
+					(size 1.27 1.27)
+				)
+				(hide yes)
+			)
+		)
+		(property "Package" ""
 			(at 247.65 36.83 0)
 			(effects
@@
 			)
 		)
-		(pin "MP"
+		(pin "1"
 		)
 		(instances
